File: PCIE x1 to MXM3.0/PCIEx1toMXM3.0.kicad_pcb (KiCad board)
At the start: 2 copper layers, 100 x 93.2 mm, 35 parts, among them J1 Bus_PCI_Express_x1, J2 MXM3.0, J3 208658-1081, J4 45558-0003, J6 PinHeader_1x4_P2mm_Drill1mm, Q1 BC848, SW1 SW_Slide_1P2T_CK_OS102011MS2Q, SW2 SW_Slide_1P2T_CK_OS102011MS2Q, U1 AMS1117-5.0

Commit message: Fixed minor issues
Parts:
- removed D6: 1N4007, Diode_THT:D_DO-41_SOD81_P10.16mm_Horizontal
Connections:
- J4 pad 1: Net-(D6-Pad2) -> +12V
- J4 pad 2: Net-(D6-Pad2) -> +12V
- J4 pad 3: Net-(D6-Pad2) -> +12V
Routing:
- net +12V: track 288.6 -> 335.9 mm, vias 11 -> 10
- net Net-(D6-Pad2): track 22.7 -> 0.00 mm
- net GND: track 187.2 -> 206.8 mm, vias 26 -> 46
