File: PCIE x16 to MXM3.0/PCIEx16toMXM3.0.sch (KiCad schematic (older format))
At the start: 42 parts, among them J1 Bus_PCI_Express_x16, J2 MXM3.0, J3 HDMI_A_1.4, J4 2040210-1_NonStock, J5 74320-9010, U1 AMS1117-5.0

Commit message: Started work on x16 adapter
Parts:
- removed D1, D5: 1N4007, Diode_THT:D_DO-41_SOD81_P10.16mm_Horizontal, symbol Diode:1N4007
- removed D2, D4: LED, symbol Device:LED
- removed J1: Bus_PCI_Express_x16, Connector_PCBEdge:BUS_PCIexpress_x16, symbol Connector1:Bus_PCI_Express_x16
- removed J3: HDMI_A_1.4, symbol Connector:HDMI_A_1.4
- removed J5: 74320-9010, digikey-footprints:DVI_Female_74320-9010, symbol dk_USB-DVI-HDMI-Connectors:74320-9010
- removed R2, R4: R_US, symbol Device:R_US
- added C15, C17: 22μF, symbol Device:C
- added C16: 0.1μF 16V, symbol Device:C_Small
- added D1, D5, D7: PMEG4010ET, Diode_SMD:D_SOT-23_ANK, symbol Diode:PMEG4010ET
- added J1: Bus_PCI_Express_x16, Connector_PCBEdge:BUS_PCIexpress_x16, symbol Connector:Bus_PCI_Express_x16
- added J3: 208658-1081, 2086581081, symbol SamacSys_Parts:208658-1081
- added J4: 45558-0003, 455580003, symbol SamacSys_Parts:45558-0003
- added L1: 4.7μH, symbol Device:L
- added Q1: BC848, Package_TO_SOT_SMD:SOT-23, symbol Transistor_BJT:BC848
- added R12: 75Ω, symbol Device:R_US
- added R14, R18: 4.3KΩ, symbol Device:R_US
- added R15, R17: 100KΩ, symbol Device:R_US
- added R16, R20: 2.2KΩ, symbol Device:R_US
- added SW1, SW2: SW_SPST, symbol Switch:SW_SPST
- C1, C2: value C -> 100μF
- C14, C3: value C -> 22μF
- FB1, FB2, FB3, FB4, FB5: symbol dk_Ferrite-Beads-and-Chips:BLM18PG121SN1D -> PCIEx1toMXM3.0-rescue:BLM18PG121SN1D-dk_Ferrite-Beads-and-Chips
- J5: renamed from J4; symbol dk_USB-DVI-HDMI-Connectors:2040210-1_NonStock -> PCIEx1toMXM3.0-rescue:2040210-1_NonStock-dk_USB-DVI-HDMI-Connectors
- R1: value R_US -> 1KΩ
- R3: value R_US -> 2KΩ
- R6: value 10K -> 100K
- gave numbers to parts that had none: 1
Connections:
- net PWR_EN is gone; now on net Enable: J2.8 (PWR_EN)
- net +12V: now also D1.2 (A), D7.2 (A), J1.A2 (+12V), J1.A3 (+12V), J1.B1 (+12V), J1.B2 (+12V), J1.B3 (+12V), J4.1, J4.2, J4.3
- net +3V3: now also C15.1, C17.1, J1.A10 (+3.3V), J1.A9 (+3.3V), J1.B8 (+3.3V), R14.1, R16.1, R18.2, R20.2
- net +5V: now also J3.18 (+5V), L1.2; no longer C14.1, C3.1
- net C1: now also R12.1
- net CEC: now also J3.13 (CEC)
- net GND: now also C14.1, C3.1, J6.1 (-), R1.1, C15.2, C16.2, C17.2, J1.A12 (GND), J1.A15 (GND), J1.A18 (GND), J1.A20 (GND), J1.A23 (GND), J1.A24 (GND), J1.A27 (GND), J1.A28 (GND), J1.A31 (GND), J1.A34 (GND), J1.A37 (GND), J1.A38 (GND), J1.A4 (GND), J1.A41 (GND), J1.A42 (GND), J1.A45 (GND), J1.A46 (GND), J1.A49 (GND), J1.A51 (GND), J1.A54 (GND), J1.A55 (GND), J1.A58 (GND), J1.A59 (GND), J1.A62 (GND), J1.A63 (GND), J1.A66 (GND), J1.A67 (GND), J1.A70 (GND), J1.A71 (GND), J1.A74 (GND), J1.A75 (GND), J1.A78 (GND), J1.A79 (GND), J1.A82 (GND), J1.B13 (GND), J1.B16 (GND), J1.B18 (GND), J1.B21 (GND), J1.B22 (GND), J1.B25 (GND), J1.B26 (GND), J1.B29 (GND), J1.B32 (GND), J1.B35 (GND), J1.B36 (GND), J1.B39 (GND), J1.B4 (GND), J1.B40 (GND), J1.B43 (GND), J1.B44 (GND), J1.B47 (GND), J1.B49 (GND), J1.B52 (GND), J1.B53 (GND), J1.B56 (GND), J1.B57 (GND), J1.B60 (GND), J1.B61 (GND), J1.B64 (GND), J1.B65 (GND), J1.B68 (GND), J1.B69 (GND), J1.B7 (GND), J1.B72 (GND), J1.B73 (GND), J1.B76 (GND), J1.B77 (GND), J1.B80 (GND), J3.11 (CKS), J3.17 (GND), J3.2 (D2S), J3.5 (D1S), J3.8 (D0S), J3.MH1, J3.MH2, J3.MH3, J3.MH4, J4.4, J4.5, J4.6, SW1.2 (B), SW2.2 (B); no longer C14.2, C3.2, R1.2
- net PER0_N: now also J1.A17 (PERn0)
- net PER0_P: now also J1.A16 (PERp0)
- net PER10_N: now also J1.A61 (PERn10)
- net PER10_P: now also J1.A60 (PERp10)
- net PER11_N: now also J1.A65 (PERn11)
- net PER11_P: now also J1.A64 (PERp11)
- net PER12_N: now also J1.A69 (PERn12)
- net PER12_P: now also J1.A68 (PERp12)
- net PER13_N: now also J1.A73 (PERn13)
- net PER13_P: now also J1.A72 (PERp13)
- net PER14_N: now also J1.A77 (PERn14)
- net PER14_P: now also J1.A76 (PERp14)
- net PER15_N: now also J1.A81 (PERn15)
- net PER15_P: now also J1.A80 (PERp15)
- net PER1_N: now also J1.A22 (PERn1)
- net PER1_P: now also J1.A21 (PERp1)
- net PER2_N: now also J1.A26 (PERn2)
- net PER2_P: now also J1.A25 (PERp2)
- net PER3_N: now also J1.A30 (PERn3)
- net PER3_P: now also J1.A29 (PERp3)
- net PER4_N: now also J1.A36 (PERn4)
- net PER4_P: now also J1.A35 (PERp4)
- net PER5_N: now also J1.A40 (PERn5)
- net PER5_P: now also J1.A39 (PERp5)
- net PER6_N: now also J1.A44 (PERn6)
- net PER6_P: now also J1.A43 (PERp6)
- net PER7_N: now also J1.A48 (PERn7)
- net PER7_P: now also J1.A47 (PERp7)
- net PER8_N: now also J1.A53 (PERn8)
- net PER8_P: now also J1.A52 (PERp8)
- net PER9_N: now also J1.A57 (PERn9)
- net PER9_P: now also J1.A56 (PERp9)
- net PERST: now also J1.A11 (~PERST), Q1.2 (E)
- net PET0_N: now also J1.B15 (PETn0)
- net PET0_P: now also J1.B14 (PETp0)
- net PET10_N: now also J1.B59 (PETn10)
- net PET10_P: now also J1.B58 (PETp10)
- net PET11_N: now also J1.B63 (PETn11)
- net PET11_P: now also J1.B62 (PETp11)
- net PET12_N: now also J1.B67 (PETn12)
- net PET12_P: now also J1.B66 (PETp12)
- net PET13_N: now also J1.B71 (PETn13)
- net PET13_P: now also J1.B70 (PETp13)
- net PET14_N: now also J1.B75 (PETn14)
- net PET14_P: now also J1.B74 (PETp14)
- net PET15_N: now also J1.B79 (PETn15)
- net PET15_P: now also J1.B78 (PETp15)
- net PET1_N: now also J1.B20 (PETn1)
- net PET1_P: now also J1.B19 (PETp1)
- net PET2_N: now also J1.B24 (PETn2)
- net PET2_P: now also J1.B23 (PETp2)
- net PET3_N: now also J1.B28 (PETn3)
- net PET3_P: now also J1.B27 (PETp3)
- net PET4_N: now also J1.B34 (PETn4)
- net PET4_P: now also J1.B33 (PETp4)
- net PET5_N: now also J1.B38 (PETn5)
- net PET5_P: now also J1.B37 (PETp5)
- net PET6_N: now also J1.B42 (PETn6)
- net PET6_P: now also J1.B41 (PETp6)
- net PET7_N: now also J1.B46 (PETn7)
- net PET7_P: now also J1.B45 (PETp7)
- net PET8_N: now also J1.B51 (PETn8)
- net PET8_P: now also J1.B50 (PETp8)
- net PET9_N: now also J1.B55 (PETn9)
- net PET9_P: now also J1.B54 (PETp9)
- net TH_OVERT#: now also Q1.1 (B), R17.1
- net WAKE: now also J1.B11 (~WAKE)
- net at U1.2 (VO): now also D5.2 (A)
- net at C1.1, C2.1, U1.3 (VI): now also D1.1 (K)
- net REFCLK_N: now reaches J2.153 (PEX_REFCLK#)
- net REFCLK_N: now also J1.A14 (REFCLK-)
- net REFCLK_P: now reaches J2.155 (PEX_REFCLK)
- net REFCLK_P: now also J1.A13 (REFCLK+)
- net CK_N: now reaches J2.176 (LVDS_LCLK#)
- net CK_N: now also J3.12 (CK-)
- net CK_P: now reaches J2.178 (LVDS_LCLK)
- net CK_P: now also J3.10 (CK+)
- net D2_N: now reaches J2.188 (LVDS_LTX2#)
- net D2_N: now also J3.3 (D2-)
- net D2_P: now reaches J2.190 (LVDS_LTX2)
- net D2_P: now also J3.1 (D2+)
- net D1_N: now reaches J2.194 (LVDS_LTX1#)
- net D1_N: now also J3.6 (D1-)
- net D1_P: now reaches J2.196 (LVDS_LTX1)
- net D1_P: now also J3.4 (D1+)
- net PRSNT_R#: now reaches J2.2 (PRSNT_R#)
- net PRSNT_R#: now also R15.1
- net D0_N: now reaches J2.200 (LVDS_LTX0#)
- net D0_N: now also J3.9 (D0-)
- net D0_P: now reaches J2.202 (LVDS_LTX0)
- net D0_P: now also J3.7 (D0+)
- net VGA_DISABLE#: now reaches J2.21 (VGA_DISABLE#)
- net VGA_DISABLE#: now also SW2.1 (A)
- net TH_PWM: now reaches J2.24 (TH_PWM)
- net TH_PWM: now also J6.4 (PWM)
- net DP_A_HPD: now reaches J2.276 (DP_A_HPD), J5.18, R5.1
- net TMDS_HPD: now reaches J2.31 (DVI_HPD), R6.2
- net TMDS_HPD: now also J3.19 (HPD/HEAC-)
- net SMDAT: now reaches J2.32 (SMB_DAT)
- net SMDAT: now also J1.B6 (SMDAT), R20.1
- net TMDS_SDA: now reaches J2.33 (LVDS_DDC_DAT)
- net TMDS_SDA: now also J3.16 (SDA), R14.2
- net SMCLK: now reaches J2.34 (SMB_CLK)
- net SMCLK: now also J1.B5 (SMCLK), R16.2
- net TMDS_SCL: now reaches J2.35 (LVDS_DDC_CLK)
- net TMDS_SCL: now also J3.15 (SCL), R18.1
- net Enable: now reaches D3.2 (A), R3.2
- net Enable: now also R1.2, C16.1
- net at J6.2 (+): now also D7.1 (K)
- net DP_A_L0_P: now reaches C12.2, J5.1
- net DP_A_L3_P: now reaches C6.2, J5.10
- net DP_A_L3_N: now reaches C7.2, J5.12
- net DP_A_AUX_P: now reaches C4.2, J5.15
- net DP_A_AUX_N: now reaches C5.2, J5.17
- net DP_A_L0_N: now reaches C13.2, J5.3
- net DP_A_L1_P: now reaches C10.2, J5.4
- net DP_A_L1_N: now reaches C11.2, J5.6
- net DP_A_L2_P: now reaches C8.2, J5.7
- net DP_A_L2_N: now reaches C9.2, J5.9
- new net: C14.2, C3.2, D5.1 (K), L1.1
- new net: J1.A1 (~PRSNT1), J1.B17 (~PRSNT2)
- new net: R12.2, SW1.1 (A)
- new net +3.3VA: J1.B10 (3.3Vaux), Q1.3 (C), R15.2, R17.2
- no-connect marks 1 -> 43
Other:
- note added: "*May not need all capacitors"
- note added: "1. This model only contains (1) HDMI 1.4 Type A\nconnector and a VGA dummy toggle."
- note added: "2. SMBus lines are optional."
- note added: "3. CLKREQ is optional."
- note added: "4. You may ignore some of the diodes.\n They are for protection."
- note added: "5V"
- note added: "5V status LED"
- note added: "Available for LVDS/TMDS output testing and for usage as a display device."
- note added: "Cooling Fan Circuit"
- note added: "Displayport Connector 0"
- note added: "Fake presence of 1 display\n"
- note added: "HDMI Port 0 (TMDS)"
- note added: "No pin to plug tachometer in, it seems."
- note added: "Notes:"
- note added: "Optional, and will likely be omitted."
- note added: "PCIE 6 Pin Power"
- note added: "PCIE Device Mode Switch"
- note added: "PCIE x1 to MXM 3.0 adapter for basic use."
- note added: "Power control"
- note added: "Signals when 5V power is available.\nPWR_EN can be asserted when 5V\nrail is on and stablized."
- note added: "Thermal shutdown is required. Send a \nPCIE reset signal when TH_OVERT# is\nhigh to prevent damage to MXM module."
- note added: "This HDMI port is optional for the test board,\nit doesn't have any protection features and likely\ndoesn't work that well but it's there if needed."
- note added: "This external power input is \noptional. Traces need to be large, \nand protection is recommended,\nbut not needed."
- note added: "VGA Compatible / 3D Render Device"
- note added: "VGA Dummy Toggle"
- note removed: "Displayport Connector type A"
- note removed: "Power status LEDs"
- moved on the sheet: C2, C3, D3, FB1, FB2, FB3, FB4, FB5, J6, R10, R11, R3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
