File: PCIE x16 to MXM3.0 Mini/PCIEx16toMXM3.0 Mini.kicad_pcb (KiCad board)
At the start: 4 copper layers, 336.5 x 112.5 mm, 20 parts, among them J1 Bus_PCI_Express_x16, J2 MXM3.0, J3 208658-1081, J4 45558-0003, Q1 BC848, U1 AMS1117-5.0

Commit message: Made some changes
Parts:
- added REF**: MountingHole_3.2mm_M3_Pad, MountingHole:MountingHole_3.2mm_M3_Pad, F.Cu at (7.81, 5.17)
- added REF**: MOLEX_47272-0001, PCIEtoMXM:MOLEX_47272-0001, F.Cu at (0.00, 21.0)
- added REF**: MOLEX_47272-0001, PCIEtoMXM:MOLEX_47272-0001, F.Cu at (0.00, 69.5)
- added REF**: MOLEX_47272-0001, PCIEtoMXM:MOLEX_47272-0001, F.Cu at (0.00, 92.0)
- added REF**: MountingHole_3.2mm_M3_Pad, MountingHole:MountingHole_3.2mm_M3_Pad, F.Cu at (7.00, 103.7)
- moved J4 193.3 mm to (133.5, 3.17)
- moved J3 191.4 mm to (6.08, 46.5)
- moved MH3 182.8 mm to (36.3, 22.9)
- moved MH4 182.8 mm to (111.4, 22.9)
- moved J2 182.8 mm to (73.9, 87.9)
Routing:
- net /PER15_P: track 0.00 -> 51.3 mm, vias 0 -> 1
- net /PER15_N: track 0.00 -> 51.3 mm, vias 0 -> 1
- net /PER14_N: track 0.00 -> 46.9 mm, vias 0 -> 1
- net /PER14_P: track 0.00 -> 46.9 mm, vias 0 -> 1
- net /PER13_N: track 0.00 -> 45.5 mm, vias 0 -> 1
- net /PER13_P: track 0.00 -> 45.5 mm, vias 0 -> 1
- net /PET15_P: track 0.00 -> 45.0 mm
- net /PET15_N: track 0.00 -> 45.0 mm
- net /PER12_P: track 0.00 -> 43.3 mm, vias 0 -> 1
- net /PER12_N: track 0.00 -> 43.3 mm, vias 0 -> 1
- net /PET14_P: track 0.00 -> 42.3 mm
- net /PET14_N: track 0.00 -> 42.3 mm
- net /PER11_P: track 0.00 -> 41.0 mm, vias 0 -> 1
- net /PER11_N: track 0.00 -> 41.0 mm, vias 0 -> 1
- net /PET13_P: track 0.00 -> 39.5 mm
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Other:
- board size 336.5 x 112.5 mm -> 339.7 x 112.5 mm

Commit message: Made some changes
Parts:
- removed the REF** at (-186.1, 108.3)
- removed the REF** at (-186.2, 18.0)
- moved D1 169.0 mm to (128.4, 23.0)
- moved D1 168.6 mm to (131.2, 89.8)
- moved D5 168.6 mm to (131.4, 83.0)
- moved D5 168.6 mm to (132.5, 23.0)
- moved D7 168.6 mm to (136.9, 23.0)
- moved FB1 168.6 mm to (136.7, 70.9)
- moved FB2 168.6 mm to (136.5, 76.5)
- moved FB3 168.6 mm to (136.5, 65.2)
- moved FB4 168.6 mm to (135.7, 38.3)
- moved FB5 168.6 mm to (139.3, 33.7)
- moved Q1 168.6 mm to (141.4, 23.0)
- moved U1 168.6 mm to (137.5, 54.1)
- renumbered REF** to MH1
Routing:
- net +12V: track 0.00 -> 252.6 mm, vias 0 -> 7
- net /SMDAT: track 0.00 -> 64.3 mm, vias 0 -> 2
- net /SMCLK: track 0.00 -> 63.8 mm, vias 0 -> 2
- net +3V3: track 0.00 -> 41.0 mm, vias 0 -> 2
- net Net-(J1-PadA1): track 0.00 -> 25.8 mm, vias 0 -> 3
- net /PET2_P: track 0.00 -> 16.1 mm
- net /PET2_N: track 0.00 -> 16.1 mm
Other:
- board size 339.7 x 112.5 mm -> 148 x 108.2 mm

Commit message: Made some changes
Parts:
- D1, D5: value 1N4007 -> PMEG4010ET
- J4: value 45558-0003 -> Molex-45586 8 Pin PWR; footprint 455580003 -> PCIEtoMXM:Molex_45586-8-Pin-PWR
- J5: renamed from REF**; value MOLEX_47272-0001 -> 47272-0001
- J6: renamed from REF**; value MOLEX_47272-0001 -> Fan_4pin
- moved J4 7.84 mm to (138.0, 9.60)
- moved D1 4.85 mm to (130.5, 27.4)
- moved D5 4.85 mm to (134.6, 27.4)
- moved Q1 4.85 mm to (143.5, 27.4)
- moved D7 4.85 mm to (139.1, 27.4)
- moved J7 3.00 mm to (0.00, 24.0)
- moved MH2 2.82 mm to (5.00, 5.00)
- moved J3 2.02 mm to (4.08, 46.8)
- renumbered REF** to J7, REF** to MH2
Connections:
- net Net-(C10-Pad1) renamed /DP_A_L1_P
- net Net-(C11-Pad1) renamed /DP_A_L1_N
- net Net-(C12-Pad1) renamed /DP_A_L0_P
- net Net-(C13-Pad1) renamed /DP_A_L0_N
- net Net-(C4-Pad1) renamed /DP_A_AUX_P
- net Net-(C5-Pad1) renamed /DP_A_AUX_N
- net Net-(C7-Pad1) renamed /DP_A_L3_N
- net Net-(C8-Pad1) renamed /DP_A_L2_P
- net Net-(C9-Pad1) renamed /DP_A_L2_N
- net Net-(J2-Pad199) renamed /DP_C_L0#
- net Net-(J2-Pad201) renamed /DP_C_L0
- net Net-(J2-Pad205) renamed /DP_C_L1#
- net Net-(J2-Pad207) renamed /DP_C_L1
- net Net-(J2-Pad211) renamed /DP_C_L2#
- net Net-(J2-Pad213) renamed /DP_C_L2
- net Net-(J2-Pad217) renamed /DP_C_L3#
- net Net-(J2-Pad219) renamed /DP_C_L3
- net Net-(J2-Pad223) renamed /DP_C_AUX#
- net Net-(J2-Pad225) renamed /DP_C_AUX
- net Net-(J2-Pad246) renamed /DP_B_L0#
- net Net-(J2-Pad248) renamed /DP_B_L0
- net Net-(J2-Pad252) renamed /DP_B_L1#
- net Net-(J2-Pad254) renamed /DP_B_L1
- net Net-(J2-Pad258) renamed /DP_B_L2#
- net Net-(J2-Pad260) renamed /DP_B_L2
- net Net-(J2-Pad264) renamed /DP_B_L3#
- net Net-(J2-Pad266) renamed /DP_B_L3
- net Net-(J2-Pad270) renamed /DP_B_AUX#
- net Net-(J2-Pad272) renamed /DP_B_AUX
- D5 pad 1: +5V -> Net-(C14-Pad2)
- J1 pad B12: Net-(J1-PadB12) -> /CLKREQ#
- J1 pad B31: Net-(J1-PadB31) -> Net-(J1-PadA1)
- J1 pad B48: Net-(J1-PadB48) -> Net-(J1-PadA1)
- J1 pad B81: Net-(J1-PadB81) -> Net-(J1-PadA1)
- J2 pad 154: Net-(J2-Pad154) -> /CLKREQ#
- J2 pad 206: /DP_D_L3# -> /DP_D_L0#
- J2 pad 208: /DP_D_L3 -> /DP_D_L0
- J2 pad 212: /DP_D_L3# -> /DP_D_L1#
- J2 pad 214: /DP_D_L3 -> /DP_D_L1
- J2 pad 218: /DP_D_L3# -> /DP_D_L2#
- J2 pad 220: /DP_D_L3 -> /DP_D_L2
- J2 pad 234: Net-(J2-Pad234) -> /DP_C_HPD
- J2 pad 273: Net-(C6-Pad1) -> /DP_A_HPD
- J2 pad 274: Net-(J2-Pad274) -> /DP_C_HPD
- J2 pad MP: GND -> (no net)
- J4 pad 4: GND -> +12V
- J5 pad 1: (no net) -> Net-(C20-Pad2)
- J5 pad 10: (no net) -> Net-(C4-Pad2)
- J5 pad 11: (no net) -> GND
- J5 pad 12: (no net) -> Net-(C24-Pad1)
- J5 pad 13: (no net) -> Net-(J5-Pad13)
- J5 pad 14: (no net) -> Net-(J5-Pad14)
- J5 pad 15: (no net) -> Net-(C26-Pad1)
- J5 pad 16: (no net) -> GND
- J5 pad 17: (no net) -> Net-(C25-Pad1)
- J5 pad 18: (no net) -> /DP_A_HPD
- J5 pad 19: (no net) -> GND
- J5 pad 2: (no net) -> GND
- J5 pad 20: (no net) -> +3V3
- J5 pad 3: (no net) -> Net-(C23-Pad1)
- J5 pad 4: (no net) -> Net-(C19-Pad2)
- J5 pad 5: (no net) -> GND
- J5 pad 6: (no net) -> Net-(C22-Pad1)
- J5 pad 7: (no net) -> Net-(C18-Pad2)
- J5 pad 8: (no net) -> GND
- J5 pad 9: (no net) -> Net-(C21-Pad1)
- J5 pad S1: (no net) -> GND
- J5 pad S2: (no net) -> GND
- J5 pad S3: (no net) -> GND
- J5 pad S4: (no net) -> GND
- J6 pad 1: (no net) -> GND
- J6 pad 2: (no net) -> Net-(D7-Pad1)
- J6 pad 3: (no net) -> Net-(J6-Pad3)
- J6 pad 4: (no net) -> TH_PWM
Routing:
- net +12V: track 252.6 -> 353.4 mm, vias 7 -> 8
- net /REFCLK_P: track 0.00 -> 50.0 mm, vias 0 -> 1
- net /REFCLK_N: track 0.00 -> 50.0 mm, vias 0 -> 1
- net /PET3_P: track 16.1 -> 49.8 mm
- net /PET3_N: track 16.1 -> 49.8 mm
- net /PET2_P: track 16.1 -> 49.7 mm
- net /PET2_N: track 16.1 -> 49.7 mm
- net /PET1_P: track 16.9 -> 50.0 mm
- net /PET1_N: track 16.9 -> 50.0 mm
- net /PET4_P: track 17.9 -> 49.7 mm
- net /PET4_N: track 17.9 -> 49.6 mm
- net /PET0_N: track 18.3 -> 50.0 mm
- net /PET0_P: track 18.3 -> 50.0 mm
- net /PET6_P: track 21.0 -> 49.9 mm
- net /PET6_N: track 21.0 -> 49.9 mm
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
Commit message: Made some changes and added new Altium documents
Parts:
- added J6: 47272-0001, PCIEtoMXM:MOLEX_47272-0001, F.Cu at (0.00, 46.8)
- J5: renamed from J6; value Fan_4pin -> 47272-0001
- moved J2 8.87 mm to (82.3, 85.2)
- moved MH3 8.87 mm to (44.8, 20.2)
- moved MH4 8.87 mm to (119.8, 20.2)
- renumbered J4 to J3, J5 to J4, J3 to J8
Connections:
- MH1 pad 1: (no net) -> GND
- MH2 pad 1: (no net) -> GND
Routing:
- net +12V: track 353.4 -> 0.00 mm, vias 8 -> 0
- net /SMDAT: track 64.3 -> 0.00 mm, vias 2 -> 0
- net /SMCLK: track 63.8 -> 0.00 mm, vias 2 -> 0
- net +3V3: track 41.0 -> 0.00 mm, vias 2 -> 0
- net /PER4_P: track 50.0 -> 27.6 mm
- net /PER4_N: track 50.0 -> 27.6 mm
- net /PER5_P: track 50.0 -> 27.8 mm
- net /PER5_N: track 50.0 -> 27.8 mm
- net /PER6_P: track 49.9 -> 28.5 mm
- net /PER6_N: track 49.9 -> 28.5 mm
- net /PER7_N: track 50.0 -> 29.6 mm
- net /PER7_P: track 50.0 -> 29.6 mm
- net /PER3_P: track 49.7 -> 29.5 mm
- net /PER3_N: track 49.7 -> 29.5 mm
- net /PER2_P: track 49.5 -> 29.7 mm
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- added copper zone on In1.Cu, net GND
