File: PCIE x16 to MXM3.0 Mini/PCIEx16toMXM3.0 Mini.sch (KiCad schematic (older format))
At the start: 53 parts, among them J1 Bus_PCI_Express_x16, J2 MXM3.0, J3 208658-1081, J4 45558-0003, J5 2040210-1_NonStock, J6 Fan_4pin, Q1 BC848, SW1 SW_SPST, SW2 SW_SPST, U1 AMS1117-5.0

Commit message: Made some changes
Parts:
- added C18, C19, C20, C21, C22, C23, C24, C25, C26: 0.1μF 16V, symbol Device:C_Small
- added C27, C29, C31, C33, C35, C36, C38, C40, C42, C44, C46, C48, C50, C52, C54, C56, C58: 0.22μF 6.3V, symbol Device:C_Small
- added C28, C30, C32, C34, C37, C39, C41, C43, C45, C47, C49, C51, C53, C55, C57, C59: (no value), symbol Device:C_Small
- added J7: 47272-0001, MOLEX_47272-0001, symbol MolexDisplayport:47272-0001
- added R13: 100K, symbol Device:R_US
- added R19, R4: 1MΩ, symbol Device:R_US
- C4: value 0.1uF -> 0.1μF 16V; symbol Device:C -> Device:C_Small
Connections:
- net labels added: CLKREQ#, DP_B_AUX, DP_B_AUX#, DP_B_L0, DP_B_L0#, DP_B_L1, DP_B_L1#, DP_B_L2, DP_B_L2#, DP_B_L3, DP_B_L3#, DP_C_AUX, DP_C_AUX#, DP_C_HPD, DP_C_L0, DP_C_L0#, DP_C_L1, DP_C_L1#, DP_C_L2, DP_C_L2#, DP_C_L3, DP_C_L3#, DP_D_L0, DP_D_L0#, DP_D_L1, DP_D_L1#, DP_D_L2, DP_D_L2#, GNDD
- wire segments 357 -> 471
- no-connect marks 43 -> 49
Other:
- note added: "*Omit"
- note added: "1. This model only contains (1) HDMI 1.4 Type A\nconnector and 3 DisplayPort Type A ports."
- note added: "4. Protection diodes are not present."
- note added: "5. VGA_Disable switch is not necessary."
- note added: "Available for DP display device."
- note added: "Available for LVDS/TMDS display device."
- note added: "DisplayPort Port 0"
- note added: "PCIE x16 to MXM 3.0 Mini Adapter"
- note added: "This DisplayPort port is not designed\nwith ESD protection circuitry in mind."
- note added: "This HDMI port is not designed\nwith ESD protection circuitry in mind."
- note removed: "1. This model only contains (1) HDMI 1.4 Type A\nconnector and a VGA dummy toggle."
- note removed: "4. You may ignore some of the diodes.\n They are for protection."
- note removed: "Available for LVDS/TMDS output testing and for usage as a display device."
- note removed: "PCIE x1 to MXM 3.0 adapter for basic use."
- note removed: "This HDMI port is optional for the test board,\nit doesn't have any protection features and likely\ndoesn't work that well but it's there if needed."
- moved on the sheet: C10, C11, C12, C13, C4, C5, C6, C7, C8, C9, J3, J5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

Commit message: Made some changes
Parts:
- removed C36: 0.22μF 6.3V, symbol Device:C_Small
- renumbered J7 to J5, J5 to J99
Connections:
- wire segments 471 -> 459
Other:
- moved on the sheet: C15, C17, C27, C28, C29, C30, C31, C32, C33, C34, C35, C37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

Commit message: Made some changes and added new Altium documents
Parts:
- renumbered J4 to J3
Changed lines of the file:
@@
 4. Protection diodes are not present.
 $Comp
-L SamacSys_Parts:45558-0003 J4
+L SamacSys_Parts:45558-0003 J3
 U 1 1 621FF001
 P 12650 7000
-F 0 "J4" H 13050 7265 50  0000 C CNN
+F 0 "J3" H 13050 7265 50  0000 C CNN
 F 1 "45558-0003" H 13050 7174 50  0000 C CNN
 F 2 "455580003" H 13300 7100 50  0001 L CNN
@@
 Connection ~ 5050 2950
 Connection ~ 5150 3050
+$Sheet
+S 800  2850 1750 1400
+U 60999EC8
+F0 "Page_PCIE" 50
+F1 "Page_PCIE.sch" 50
+$EndSheet
 Wire Bus Line
 	12550 3550 13300 3550
@@
 Wire Bus Line
 	7000 3550 12550 3550
-$Sheet
-S 800  2850 1750 1400
-U 60999EC8
-F0 "Page_PCIE" 50
-F1 "Page_PCIE.sch" 50
-$EndSheet
 $EndSCHEMATC
